Commit message: world_ws13: 重构 BaseMoveController, 优化遮挡处理与 PID 控制
变更内容:
  - [新增] BaseMoveController.cpp/h: 重构基础运动控制器
  - [新增] change_data.py: 数据格式转换脚本
  - [新增] 01_400.txt / label_400.txt: 更新标注数据集
  - [移除] basemove2.cpp: 被 BaseMoveController 替代
  - [移除] label_100.txt / label_150.txt: 旧版标注数据
  - [优化] occlusion_handing 遮挡处理算法
  - [优化] PID.cpp 控制器参数
  - [优化] zbuffer_func 主节点性能
  - [文档] README.md: 更新版本迭代日志

File: src/zwei/map1_add/urdf/map_110.urdf (robot description, URDF)
Before this commit: robot zwei, 27 links, 26 joints
Links:
- removed link Link30
- removed link Link32
- removed link Link36
- added link Link25, mass 42.8749999999999; collision mesh filename=package://zwei/meshes/Link25.STL; visual mesh filename=package://zwei/meshes/r102.dae
- added link Link27, mass 42.8749999999999; collision mesh filename=package://zwei/meshes/Link27.STL; visual mesh filename=package://zwei/meshes/r316.dae
- added link Link31, mass 42.875; collision mesh filename=package://zwei/meshes/Link31.STL; visual mesh filename=package://zwei/meshes/r705.dae
- link Link28: geometry collision mesh filename=package://zwei/meshes/Link28.STL; visual mesh filename=package://zwei/meshes/r406.dae
- link Link33: geometry collision mesh filename=package://zwei/meshes/Link33.STL; visual mesh filename=package://zwei/meshes/r928.dae
- link Link34: geometry collision mesh filename=package://zwei/meshes/Link34.STL; visual mesh filename=package://zwei/meshes/ra01.dae
- link Link35: geometry collision mesh filename=package://zwei/meshes/Link35.STL; visual mesh filename=package://zwei/meshes/rb01.dae
Joints:
- removed joint 30
- removed joint 32
- removed joint 36
- added joint 25: type fixed, parent base_link, child Link25, origin xyz=1.8 3.8 0.4098 rpy=1.5707963267949 0 0, axis 0 0 0
- added joint 27: type fixed, parent base_link, child Link27, origin xyz=4.2 3.8 0.399800000000001 rpy=1.5707963267949 0 0, axis 0 0 0
- added joint 31: type fixed, parent base_link, child Link31, origin xyz=1.8 6.2 0.7398 rpy=-1.5707963267949 0 3.14159265358979, axis 0 0 0

File: src/zwei/map1_add/urdf/map_111.urdf (robot description, URDF)
Before this commit: robot zwei, 27 links, 26 joints
Links:
- removed link Link25
- removed link Link27
- removed link Link29
- added link Link28, mass 42.875; collision mesh filename=package://zwei/meshes/Link28.STL; visual mesh filename=package://zwei/meshes/r401.dae
- added link Link30, mass 42.875; collision mesh filename=package://zwei/meshes/Link30.STL; visual mesh filename=package://zwei/meshes/r604.dae
- added link Link32, mass 42.875; collision mesh filename=package://zwei/meshes/Link32.STL; visual mesh filename=package://zwei/meshes/r815.dae
- link Link26: geometry collision mesh filename=package://zwei/meshes/Link26.STL; visual mesh filename=package://zwei/meshes/r203.dae
- link Link31: geometry collision mesh filename=package://zwei/meshes/Link31.STL; visual mesh filename=package://zwei/meshes/r713.dae
- link Link36: geometry collision mesh filename=package://zwei/meshes/Link36.STL; visual mesh filename=package://zwei/meshes/rc20.dae
Joints:
- removed joint 25
- removed joint 27
- removed joint 29
- added joint 28: type fixed, parent base_link, child Link28, origin xyz=1.635 5 0.3748 rpy=1.5707963267949 1.5707963267949 0, axis 0 0 0
- added joint 30: type fixed, parent base_link, child Link30, origin xyz=4.025 5 0.7748 rpy=1.5707963267949 1.5707963267949 0, axis 0 0 0
- added joint 32: type fixed, parent base_link, child Link32, origin xyz=3 6.2 0.9498 rpy=-1.5707963267949 0 3.14159265358979, axis 0 0 0

File: src/zwei/map1_add/urdf/map_112.urdf (robot description, URDF)
Before this commit: robot zwei, 27 links, 26 joints
Links:
- removed link Link27
- removed link Link29
- added link Link31, mass 42.875; collision mesh filename=package://zwei/meshes/Link31.STL; visual mesh filename=package://zwei/meshes/r701.dae
- added link Link34, mass 42.875; collision mesh filename=package://zwei/meshes/Link34.STL; visual mesh filename=package://zwei/meshes/ra03.dae
- link Link25: geometry collision mesh filename=package://zwei/meshes/Link25.STL; visual mesh filename=package://zwei/meshes/r109.dae
- link Link26: geometry collision mesh filename=package://zwei/meshes/Link26.STL; visual mesh filename=package://zwei/meshes/r215.dae
- link Link32: geometry collision mesh filename=package://zwei/meshes/Link32.STL; visual mesh filename=package://zwei/meshes/r808.dae
- link Link33: geometry collision mesh filename=package://zwei/meshes/Link33.STL; visual mesh filename=package://zwei/meshes/r923.dae
- link Link35: geometry collision mesh filename=package://zwei/meshes/Link35.STL; visual mesh filename=package://zwei/meshes/rb01.dae
Joints:
- removed joint 27
- removed joint 29
- added joint 31: type fixed, parent base_link, child Link31, origin xyz=1.8 6.2 0.7398 rpy=-1.5707963267949 0 3.14159265358979, axis 0 0 0
- added joint 34: type fixed, parent base_link, child Link34, origin xyz=1.8 7.4 0.199800000000001 rpy=1.5707963267949 0 0, axis 0 0 0

File: src/zwei/map1_add/urdf/map_113.urdf (robot description, URDF)
Before this commit: robot zwei, 27 links, 26 joints
Links:
- removed link Link33
- removed link Link34
- added link Link27, mass 42.8749999999999; collision mesh filename=package://zwei/meshes/Link27.STL; visual mesh filename=package://zwei/meshes/r301.dae
- added link Link31, mass 42.875; collision mesh filename=package://zwei/meshes/Link31.STL; visual mesh filename=package://zwei/meshes/r715.dae
- link Link26: geometry collision mesh filename=package://zwei/meshes/Link26.STL; visual mesh filename=package://zwei/meshes/r229.dae
- link Link28: geometry collision mesh filename=package://zwei/meshes/Link28.STL; visual mesh filename=package://zwei/meshes/r401.dae
- link Link29: geometry collision mesh filename=package://zwei/meshes/Link29.STL; visual mesh filename=package://zwei/meshes/r513.dae
- link Link32: geometry collision mesh filename=package://zwei/meshes/Link32.STL; visual mesh filename=package://zwei/meshes/r801.dae
- link Link36: geometry collision mesh filename=package://zwei/meshes/Link36.STL; visual mesh filename=package://zwei/meshes/rc10.dae
Joints:
- removed joint 33
- removed joint 34
- added joint 27: type fixed, parent base_link, child Link27, origin xyz=4.2 3.8 0.399800000000001 rpy=1.5707963267949 0 0, axis 0 0 0
- added joint 31: type fixed, parent base_link, child Link31, origin xyz=1.8 6.2 0.7398 rpy=-1.5707963267949 0 3.14159265358979, axis 0 0 0

File: src/zwei/map1_add/urdf/map_114.urdf (robot description, URDF)
Before this commit: robot zwei, 27 links, 26 joints
Links:
- removed link Link26
- removed link Link32
- removed link Link33
- added link Link28, mass 42.875; collision mesh filename=package://zwei/meshes/Link28.STL; visual mesh filename=package://zwei/meshes/r428.dae
- added link Link29, mass 42.875; collision mesh filename=package://zwei/meshes/Link29.STL; visual mesh filename=package://zwei/meshes/r508.dae
- added link Link36, mass 42.875; collision mesh filename=package://zwei/meshes/Link36.STL; visual mesh filename=package://zwei/meshes/rc01.dae
- link Link25: geometry collision mesh filename=package://zwei/meshes/Link25.STL; visual mesh filename=package://zwei/meshes/r112.dae
- link Link27: geometry collision mesh filename=package://zwei/meshes/Link27.STL; visual mesh filename=package://zwei/meshes/r302.dae
- link Link30: geometry collision mesh filename=package://zwei/meshes/Link30.STL; visual mesh filename=package://zwei/meshes/r601.dae
- link Link31: geometry collision mesh filename=package://zwei/meshes/Link31.STL; visual mesh filename=package://zwei/meshes/r715.dae
- link Link35: geometry collision mesh filename=package://zwei/meshes/Link35.STL; visual mesh filename=package://zwei/meshes/rb01.dae
Joints:
- removed joint 26
- removed joint 32
- removed joint 33
- added joint 28: type fixed, parent base_link, child Link28, origin xyz=1.635 5 0.3748 rpy=1.5707963267949 1.5707963267949 0, axis 0 0 0
- added joint 29: type fixed, parent base_link, child Link29, origin xyz=3.165 5 0.5748 rpy=1.5707963267949 -1.5707963267949 0, axis 0 0 0
- added joint 36: type fixed, parent base_link, child Link36, origin xyz=4.2 7.4 0.549800000000001 rpy=-1.5707963267949 0 3.14159265358979, axis 0 0 0

File: src/zwei/map1_add/urdf/map_115.urdf (robot description, URDF)
Before this commit: robot zwei, 27 links, 26 joints
Links:
- removed link Link26
- removed link Link31
- removed link Link34
- added link Link27, mass 42.8749999999999; collision mesh filename=package://zwei/meshes/Link27.STL; visual mesh filename=package://zwei/meshes/r313.dae
- added link Link32, mass 42.875; collision mesh filename=package://zwei/meshes/Link32.STL; visual mesh filename=package://zwei/meshes/r801.dae
- added link Link33, mass 42.875; collision mesh filename=package://zwei/meshes/Link33.STL; visual mesh filename=package://zwei/meshes/r905.dae
- link Link25: geometry collision mesh filename=package://zwei/meshes/Link25.STL; visual mesh filename=package://zwei/meshes/r116.dae
- link Link28: geometry collision mesh filename=package://zwei/meshes/Link28.STL; visual mesh filename=package://zwei/meshes/r429.dae
- link Link30: geometry collision mesh filename=package://zwei/meshes/Link30.STL; visual mesh filename=package://zwei/meshes/r601.dae
- link Link36: geometry collision mesh filename=package://zwei/meshes/Link36.STL; visual mesh filename=package://zwei/meshes/rc12.dae
Joints:
- removed joint 26
- removed joint 31
- removed joint 34
- added joint 27: type fixed, parent base_link, child Link27, origin xyz=4.2 3.8 0.399800000000001 rpy=1.5707963267949 0 0, axis 0 0 0
- added joint 32: type fixed, parent base_link, child Link32, origin xyz=3 6.2 0.9498 rpy=-1.5707963267949 0 3.14159265358979, axis 0 0 0
- added joint 33: type fixed, parent base_link, child Link33, origin xyz=4.375 6.2 0.5748 rpy=1.5707963267949 -1.5707963267949 0, axis 0 0 0

File: src/zwei/map1_add/urdf/map_116.urdf (robot description, URDF)
Before this commit: robot zwei, 27 links, 26 joints
Links:
- removed link Link25
- removed link Link36
- added link Link29, mass 42.875; collision mesh filename=package://zwei/meshes/Link29.STL; visual mesh filename=package://zwei/meshes/r508.dae
- added link Link35, mass 42.875; collision mesh filename=package://zwei/meshes/Link35.STL; visual mesh filename=package://zwei/meshes/rb01.dae
- link Link28: geometry collision mesh filename=package://zwei/meshes/Link28.STL; visual mesh filename=package://zwei/meshes/r401.dae
- link Link30: geometry collision mesh filename=package://zwei/meshes/Link30.STL; visual mesh filename=package://zwei/meshes/r623.dae
- link Link32: geometry collision mesh filename=package://zwei/meshes/Link32.STL; visual mesh filename=package://zwei/meshes/r814.dae
- link Link33: geometry collision mesh filename=package://zwei/meshes/Link33.STL; visual mesh filename=package://zwei/meshes/r913.dae
Joints:
- removed joint 25
- removed joint 36
- added joint 29: type fixed, parent base_link, child Link29, origin xyz=3.165 5 0.5748 rpy=1.5707963267949 -1.5707963267949 0, axis 0 0 0
- added joint 35: type fixed, parent base_link, child Link35, origin xyz=2.825 7.4 0.5748 rpy=1.5707963267949 1.5707963267949 0, axis 0 0 0
