Commit message: world_ws13.5: 地图数据更新与最终优化
变更内容:
  - [优化] zbuffer_func.cpp: 主节点性能微调与稳定性改进
  - [更新] map_*.txt 地图数据集 (大规模地图数据更新)
  - [更新] flag.txt 地图标志位配置
  - [更新] wpr_simulation.zip 仿真环境包
  - [文档] README.md: 更新版本迭代日志

File: src/zwei/map1_add/urdf/map_111.urdf (robot description, URDF)
Before this commit: robot zwei, 27 links, 26 joints
Links:
- removed link Link26
- removed link Link34
- removed link Link36
- added link Link25, mass 42.8749999999999; collision mesh filename=package://zwei/meshes/Link25.STL; visual mesh filename=package://zwei/meshes/r101.dae
- added link Link27, mass 42.8749999999999; collision mesh filename=package://zwei/meshes/Link27.STL; visual mesh filename=package://zwei/meshes/r326.dae
- added link Link29, mass 42.875; collision mesh filename=package://zwei/meshes/Link29.STL; visual mesh filename=package://zwei/meshes/r501.dae
- link Link30: geometry collision mesh filename=package://zwei/meshes/Link30.STL; visual mesh filename=package://zwei/meshes/r608.dae
- link Link31: geometry collision mesh filename=package://zwei/meshes/Link31.STL; visual mesh filename=package://zwei/meshes/r716.dae
- link Link32: geometry collision mesh filename=package://zwei/meshes/Link32.STL; visual mesh filename=package://zwei/meshes/r811.dae
Joints:
- removed joint 26
- removed joint 34
- removed joint 36
- added joint 25: type fixed, parent base_link, child Link25, origin xyz=1.8 3.8 0.4098 rpy=1.5707963267949 0 0, axis 0 0 0
- added joint 27: type fixed, parent base_link, child Link27, origin xyz=4.2 3.8 0.399800000000001 rpy=1.5707963267949 0 0, axis 0 0 0
- added joint 29: type fixed, parent base_link, child Link29, origin xyz=3.165 5 0.5748 rpy=1.5707963267949 -1.5707963267949 0, axis 0 0 0

File: src/zwei/map1_add/urdf/map_112.urdf (robot description, URDF)
Before this commit: robot zwei, 27 links, 26 joints
Links:
- removed link Link25
- removed link Link26
- removed link Link31
- removed link Link33
- added link Link27, mass 42.8749999999999; collision mesh filename=package://zwei/meshes/Link27.STL; visual mesh filename=package://zwei/meshes/r308.dae
- added link Link28, mass 42.875; collision mesh filename=package://zwei/meshes/Link28.STL; visual mesh filename=package://zwei/meshes/r401.dae
- added link Link29, mass 42.875; collision mesh filename=package://zwei/meshes/Link29.STL; visual mesh filename=package://zwei/meshes/r501.dae
- added link Link30, mass 42.875; collision mesh filename=package://zwei/meshes/Link30.STL; visual mesh filename=package://zwei/meshes/r615.dae
- link Link32: geometry collision mesh filename=package://zwei/meshes/Link32.STL; visual mesh filename=package://zwei/meshes/r801.dae
- link Link34: geometry collision mesh filename=package://zwei/meshes/Link34.STL; visual mesh filename=package://zwei/meshes/ra06.dae
- link Link35: geometry collision mesh filename=package://zwei/meshes/Link35.STL; visual mesh filename=package://zwei/meshes/rb20.dae
- link Link36: geometry collision mesh filename=package://zwei/meshes/Link36.STL; visual mesh filename=package://zwei/meshes/rc16.dae
Joints:
- removed joint 25
- removed joint 26
- removed joint 31
- removed joint 33
- added joint 27: type fixed, parent base_link, child Link27, origin xyz=4.2 3.8 0.399800000000001 rpy=1.5707963267949 0 0, axis 0 0 0
- added joint 28: type fixed, parent base_link, child Link28, origin xyz=1.635 5 0.3748 rpy=1.5707963267949 1.5707963267949 0, axis 0 0 0
- added joint 29: type fixed, parent base_link, child Link29, origin xyz=3.165 5 0.5748 rpy=1.5707963267949 -1.5707963267949 0, axis 0 0 0
- added joint 30: type fixed, parent base_link, child Link30, origin xyz=4.025 5 0.7748 rpy=1.5707963267949 1.5707963267949 0, axis 0 0 0

File: src/zwei/map1_add/urdf/map_113.urdf (robot description, URDF)
Before this commit: robot zwei, 27 links, 26 joints
Links:
- removed link Link25
- removed link Link29
- added link Link30, mass 42.875; collision mesh filename=package://zwei/meshes/Link30.STL; visual mesh filename=package://zwei/meshes/r601.dae
- added link Link34, mass 42.875; collision mesh filename=package://zwei/meshes/Link34.STL; visual mesh filename=package://zwei/meshes/ra14.dae
- link Link26: geometry collision mesh filename=package://zwei/meshes/Link26.STL; visual mesh filename=package://zwei/meshes/r212.dae
- link Link27: geometry collision mesh filename=package://zwei/meshes/Link27.STL; visual mesh filename=package://zwei/meshes/r305.dae
- link Link31: geometry collision mesh filename=package://zwei/meshes/Link31.STL; visual mesh filename=package://zwei/meshes/r716.dae
- link Link32: geometry collision mesh filename=package://zwei/meshes/Link32.STL; visual mesh filename=package://zwei/meshes/r827.dae
- link Link36: geometry collision mesh filename=package://zwei/meshes/Link36.STL; visual mesh filename=package://zwei/meshes/rc01.dae
Joints:
- removed joint 25
- removed joint 29
- added joint 30: type fixed, parent base_link, child Link30, origin xyz=4.025 5 0.7748 rpy=1.5707963267949 1.5707963267949 0, axis 0 0 0
- added joint 34: type fixed, parent base_link, child Link34, origin xyz=1.8 7.4 0.199800000000001 rpy=1.5707963267949 0 0, axis 0 0 0

File: src/zwei/map1_add/urdf/map_114.urdf (robot description, URDF)
Before this commit: robot zwei, 27 links, 26 joints
Links:
- removed link Link27
- removed link Link30
- removed link Link31
- added link Link26, mass 42.875; collision mesh filename=package://zwei/meshes/Link26.STL; visual mesh filename=package://zwei/meshes/r203.dae
- added link Link32, mass 42.875; collision mesh filename=package://zwei/meshes/Link32.STL; visual mesh filename=package://zwei/meshes/r801.dae
- added link Link33, mass 42.875; collision mesh filename=package://zwei/meshes/Link33.STL; visual mesh filename=package://zwei/meshes/r914.dae
- link Link25: geometry collision mesh filename=package://zwei/meshes/Link25.STL; visual mesh filename=package://zwei/meshes/r101.dae
- link Link28: geometry collision mesh filename=package://zwei/meshes/Link28.STL; visual mesh filename=package://zwei/meshes/r401.dae
- link Link29: geometry collision mesh filename=package://zwei/meshes/Link29.STL; visual mesh filename=package://zwei/meshes/r518.dae
- link Link35: geometry collision mesh filename=package://zwei/meshes/Link35.STL; visual mesh filename=package://zwei/meshes/rb10.dae
- link Link36: geometry collision mesh filename=package://zwei/meshes/Link36.STL; visual mesh filename=package://zwei/meshes/rc15.dae
Joints:
- removed joint 27
- removed joint 30
- removed joint 31
- added joint 26: type fixed, parent base_link, child Link26, origin xyz=3 3.8 0.2098 rpy=1.5707963267949 0 0, axis 0 0 0
- added joint 32: type fixed, parent base_link, child Link32, origin xyz=3 6.2 0.9498 rpy=-1.5707963267949 0 3.14159265358979, axis 0 0 0
- added joint 33: type fixed, parent base_link, child Link33, origin xyz=4.375 6.2 0.5748 rpy=1.5707963267949 -1.5707963267949 0, axis 0 0 0

File: src/zwei/map1_add/urdf/map_115.urdf (robot description, URDF)
Before this commit: robot zwei, 27 links, 26 joints
Links:
- removed link Link28
- removed link Link36
- added link Link26, mass 42.875; collision mesh filename=package://zwei/meshes/Link26.STL; visual mesh filename=package://zwei/meshes/r201.dae
- added link Link35, mass 42.875; collision mesh filename=package://zwei/meshes/Link35.STL; visual mesh filename=package://zwei/meshes/rb01.dae
- link Link25: geometry collision mesh filename=package://zwei/meshes/Link25.STL; visual mesh filename=package://zwei/meshes/r105.dae
- link Link27: geometry collision mesh filename=package://zwei/meshes/Link27.STL; visual mesh filename=package://zwei/meshes/r301.dae
- link Link29: geometry collision mesh filename=package://zwei/meshes/Link29.STL; visual mesh filename=package://zwei/meshes/r516.dae
- link Link30: geometry collision mesh filename=package://zwei/meshes/Link30.STL; visual mesh filename=package://zwei/meshes/r603.dae
- link Link32: geometry collision mesh filename=package://zwei/meshes/Link32.STL; visual mesh filename=package://zwei/meshes/r811.dae
- link Link33: geometry collision mesh filename=package://zwei/meshes/Link33.STL; visual mesh filename=package://zwei/meshes/r917.dae
Joints:
- removed joint 28
- removed joint 36
- added joint 26: type fixed, parent base_link, child Link26, origin xyz=3 3.8 0.2098 rpy=1.5707963267949 0 0, axis 0 0 0
- added joint 35: type fixed, parent base_link, child Link35, origin xyz=2.825 7.4 0.5748 rpy=1.5707963267949 1.5707963267949 0, axis 0 0 0

File: src/zwei/map1_add/urdf/map_116.urdf (robot description, URDF)
Before this commit: robot zwei, 27 links, 26 joints
Links:
- removed link Link28
- removed link Link32
- removed link Link34
- added link Link25, mass 42.8749999999999; collision mesh filename=package://zwei/meshes/Link25.STL; visual mesh filename=package://zwei/meshes/r101.dae
- added link Link31, mass 42.875; collision mesh filename=package://zwei/meshes/Link31.STL; visual mesh filename=package://zwei/meshes/r714.dae
- added link Link36, mass 42.875; collision mesh filename=package://zwei/meshes/Link36.STL; visual mesh filename=package://zwei/meshes/rc01.dae
- link Link27: geometry collision mesh filename=package://zwei/meshes/Link27.STL; visual mesh filename=package://zwei/meshes/r303.dae
- link Link29: geometry collision mesh filename=package://zwei/meshes/Link29.STL; visual mesh filename=package://zwei/meshes/r512.dae
- link Link30: geometry collision mesh filename=package://zwei/meshes/Link30.STL; visual mesh filename=package://zwei/meshes/r601.dae
- link Link33: geometry collision mesh filename=package://zwei/meshes/Link33.STL; visual mesh filename=package://zwei/meshes/r923.dae
Joints:
- removed joint 28
- removed joint 32
- removed joint 34
- added joint 25: type fixed, parent base_link, child Link25, origin xyz=1.8 3.8 0.4098 rpy=1.5707963267949 0 0, axis 0 0 0
- added joint 31: type fixed, parent base_link, child Link31, origin xyz=1.8 6.2 0.7398 rpy=-1.5707963267949 0 3.14159265358979, axis 0 0 0
- added joint 36: type fixed, parent base_link, child Link36, origin xyz=4.2 7.4 0.549800000000001 rpy=-1.5707963267949 0 3.14159265358979, axis 0 0 0
